File: PDB/5v.kicad_sch (KiCad schematic)
At the start: 25 parts, among them M1 GENERIC_MOSFET_N, M2 GENERIC_MOSFET_N, U1 LM5116MH/NOPB

Commit message: Add 24V@1.5A
Filled 24V@1.5A schem and added hierarchal pins to each sub sheet
Parts:
- removed Iout: WB_CURRENT_LOAD, symbol TI WEBENCH:root_3_Iout_TI WEBENCH
- removed Vin: WB_BATTERY, symbol TI WEBENCH:root_3_Vin_TI WEBENCH
Connections:
- net +BATT: now reaches Cin.1, Cinx.1, M1.2 (Drain), Renable.1, Ruv2.1, U1.1 (VIN)
- net 5V@12A: now reaches Cout.1, Cout_2.1, L1.2, Rfbt.1, U1.10 (VOUT)
- net 0 renamed GND

Commit message: added fuses to each
Parts:
- added F2: TR/3216FF15-R, symbol Device:Fuse
Connections:
- net 5V@12A: now also F2.1, F2.2
Changed lines of the file:
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@@
+	(wire
+		(pts
+			(xy 427.99 138.43) (xy 427.99 140.97)
+		)
+		(stroke
+			(width 0)
+			(type default)
+		)
+	)
 	(wire
 		(pts
@@
 		(pts
 			(xy 209.55 185.42) (xy 209.55 203.2)
+		)
+		(stroke
+			(width 0)
+			(type default)
+		)
+	)
+	(wire
+		(pts
+			(xy 427.99 128.27) (xy 427.99 130.81)
 		)
 		(stroke
@@
 	(symbol
 		(lib_id "power:+1V5")
-		(at 427.99 140.97 0)
+		(at 427.99 128.27 0)
 		(unit 1)
 		(body_style 1)
@@
 		(fields_autoplaced yes)
 		(property "Reference" "#PWR029"
-			(at 427.99 144.78 0)
+			(at 427.99 132.08 0)
 			(hide yes)
 			(show_name no)
@@
 		)
 		(property "Value" "5V@12A"
-			(at 427.99 135.89 0)
+			(at 427.99 123.19 0)
 			(show_name no)
 			(do_not_autoplace no)
@@
 		)
 		(property "Footprint" ""
-			(at 427.99 140.97 0)
+			(at 427.99 128.27 0)
 			(hide yes)
 			(show_name no)
@@
 		)
 		(property "Datasheet" ""
-			(at 427.99 140.97 0)
+			(at 427.99 128.27 0)
 			(hide yes)
 			(show_name no)
@@
 		)
 		(property "Description" "Power symbol creates a global label with name \"+1V5\""
-			(at 427.99 140.97 0)
+			(at 427.99 128.27 0)
 			(hide yes)
 			(show_name no)
@@
 					(unit 1)
 				)
+			)
+		)
+	)
+	(symbol
+		(lib_id "Device:Fuse")
+		(at 427.99 134.62 180)
+		(unit 1)
+		(body_style 1)
+		(exclude_from_sim no)
+		(in_bom yes)
+		(on_board yes)
+		(in_pos_files yes)
+		(dnp no)
+		(fields_autoplaced yes)
+		(property "Reference" "F2"
+			(at 430.53 133.3499 0)
+			(show_name no)
+			(do_not_autoplace no)
+			(effects
+				(font
+					(size 1.27 1.27)
+				)
+				(justify right)
+			)
+		)
+		(property "Value" "TR/3216FF15-R"
+			(at 430.53 135.8899 0)
+			(show_name no)
+			(do_not_autoplace no)
+			(effects
+				(font
+					(size 1.27 1.27)
+				)
+				(justify right)
+			)
+		)
+		(property "Footprint" ""
+			(at 429.768 134.62 90)
+			(hide yes)
+			(show_name no)
+			(do_not_autoplace no)
+			(effects
+				(font
+					(size 1.27 1.27)
+				)
+			)
+		)
+		(property "Datasheet" ""
+			(at 427.99 134.62 0)
+			(hide yes)
+			(show_name no)
+			(do_not_autoplace no)
+			(effects
+				(font
+					(size 1.27 1.27)
+				)
+			)
+		)
+		(property "Description" "Fuse"
+			(at 427.99 134.62 0)
+			(hide yes)
+			(show_name no)
+			(do_not_autoplace no)
+			(effects
+				(font
+					(size 1.27 1.27)
+				)
+			)
+		)
+		(pin "2"
+		)
+		(pin "1"
+		)
+		(instances
+			(project "PDB"
+				(path "/a9cf05c4-aac5-4cf1-b700-1d3045f8dfbd/a24fc02a-90d5-41f1-96d5-cd0fa3bff83a"
+					(reference "F2")
+					(unit 1)
+				)

Commit message: added temp sensing on every rail available
Parts:
- added C32: 100nf, Capacitor_SMD:C_1206_3216Metric, symbol Device:C
- added R37: R_Shunt, symbol Device:R_Shunt
- added U12: INA228, Package_SO:TSSOP-10_3x3mm_P0.5mm, symbol Sensor_Energy:INA228
Connections:
- net 5V@12A: now also R37.4; no longer Cout.1, Cout_2.1, F2.1, F2.2, L1.2, Rfbt.1, U1.10 (VOUT)
- net GND: now also C32.1, U12.1 (A1), U12.2 (A0), U12.7 (GND)
- new net: Cout.1, Cout_2.1, F2.1, L1.2, Rfbt.1, U1.10 (VOUT)
- new net: F2.2, R37.1, U12.8 (Vbus)
- new net: R37.2, U12.10 (Vin+)
- new net: R37.3, U12.9 (Vin-)
- new net +3.3V: C32.2, U12.6 (VS)
- new net SCL: U12.5 (SCL)
- new net SDA: U12.4 (SDA)
- no-connect marks 0 -> 1

Commit message: added tp's, switches, inputs/outputs
Parts:
- added D15: LED, LED_SMD:LED_0805_2012Metric, symbol Device:LED
- added R42: 270, Resistor_SMD:R_1206_3216Metric_Pad1.30x1.75mm_HandSolder, symbol Device:R
- added TP4: TestPoint, TestPoint:TestPoint_Pad_D2.0mm, symbol Connector:TestPoint
Connections:
- net 5V@12A: now also R42.1, TP4.1
- net GND: now also D15.1 (K)
- new net: D15.2 (A), R42.2

Commit message: Finished all the footprints. doing poe myself now
finally.
Parts:
- C15: renamed from C32; footprint Capacitor_SMD:C_1206_3216Metric -> Capacitor_SMD:C_0603_1608Metric
- Cboot1: renamed from Cboot; footprint (none) -> Capacitor_SMD:C_0603_1608Metric
- Ccomp1: renamed from Ccomp2; footprint (none) -> Capacitor_SMD:C_0603_1608Metric
- Ccomp2: renamed from Ccomp; footprint (none) -> Capacitor_SMD:C_0603_1608Metric
- Cin1: renamed from Cin; footprint (none) -> Capacitor_SMD:C_0603_1608Metric
- Cinx1: renamed from Cinx; footprint (none) -> Capacitor_SMD:C_0603_1608Metric
- Cout1: renamed from Cout; footprint (none) -> Capacitor_SMD:C_0603_1608Metric
- Cout_1: renamed from Cout_2; footprint (none) -> Capacitor_SMD:C_0603_1608Metric
- Cramp1: renamed from Cramp; footprint (none) -> Capacitor_SMD:C_0603_1608Metric
- Css1: renamed from Css; footprint (none) -> Capacitor_SMD:C_0603_1608Metric
- Cvcc1: renamed from Cvcc; footprint (none) -> Capacitor_SMD:C_0603_1608Metric
- D12: renamed from D1; footprint (none) -> Diode_SMD:D_SOD-523
- F1: renamed from F2; footprint (none) -> Fuse:Fuse_1206_3216Metric
- L1: footprint (none) -> Inductor_SMD:L_1206_3216Metric
- M1: footprint (none) -> Package_SON:Infineon_PG-TDSON-8_6.15x5.15mm; PACKAGEREFERENCE NVMFS6H836NLT1G -> BSC117N08NS5ATMA1
- M2: footprint (none) -> Package_SON:Infineon_PG-TDSON-8_6.15x5.15mm
- R21: renamed from R37; footprint (none) -> Resistor_SMD:R_0603_1608Metric
- Rcomp1: renamed from Rcomp; footprint (none) -> Resistor_SMD:R_0603_1608Metric
- Renable1: renamed from Renable; footprint (none) -> Resistor_SMD:R_0603_1608Metric
- Rfbb1: renamed from Rfbb; footprint (none) -> Resistor_SMD:R_0603_1608Metric
- Rfbt1: renamed from Rfbt; footprint (none) -> Resistor_SMD:R_0603_1608Metric
- Rsense1: renamed from Rsense; footprint (none) -> Resistor_SMD:R_0603_1608Metric
- Rt1: renamed from Rt; footprint (none) -> Resistor_SMD:R_0603_1608Metric
- Ruv1: renamed from Ruv2; footprint (none) -> Resistor_SMD:R_0603_1608Metric
- Ruv2: renamed from Ruv1; footprint (none) -> Resistor_SMD:R_0603_1608Metric
- U8: renamed from U1; footprint (none) -> Dependencies:MXA20A_TEX
- U9: renamed from U12; footprint Package_SO:TSSOP-10_3x3mm_P0.5mm -> Package_SO:HVSSOP-10-1EP_3x3mm_P0.5mm_EP1.83x1.89mm
- renumbered D15 to D13, R42 to R22, TP4 to TP6

Commit message: fixed component footprints
Parts:
- R21: footprint Resistor_SMD:R_0603_1608Metric -> Resistor_SMD:R_Shunt_Vishay_WSR2_WSR3_KelvinConnection
Changed lines of the file:
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@@
 		(dnp no)
 		(fields_autoplaced yes)
-		(property "Reference" "#PWR024"
+		(property "Reference" "#PWR041"
 			(at 374.65 189.23 0)
 			(hide yes)
@@
 			(project "PDB"
 				(path "/a9cf05c4-aac5-4cf1-b700-1d3045f8dfbd/a24fc02a-90d5-41f1-96d5-cd0fa3bff83a"
-					(reference "#PWR024")
+					(reference "#PWR041")
 					(unit 1)
 				)
@@
 		(dnp no)
 		(fields_autoplaced yes)
-		(property "Reference" "#PWR025"
+		(property "Reference" "#PWR039"
 			(at 326.39 187.96 0)
 			(hide yes)
@@
 			(project "PDB"
 				(path "/a9cf05c4-aac5-4cf1-b700-1d3045f8dfbd/a24fc02a-90d5-41f1-96d5-cd0fa3bff83a"
-					(reference "#PWR025")
+					(reference "#PWR039")
 					(unit 1)
 				)
@@
 		(dnp no)
 		(fields_autoplaced yes)
-		(property "Reference" "#PWR054"
+		(property "Reference" "#PWR044"
 			(at 429.26 86.36 0)
 			(hide yes)
@@
 			(project "PDB"
 				(path "/a9cf05c4-aac5-4cf1-b700-1d3045f8dfbd/a24fc02a-90d5-41f1-96d5-cd0fa3bff83a"
-					(reference "#PWR054")
+					(reference "#PWR044")
 					(unit 1)
 				)
@@
 		(dnp no)
 		(fields_autoplaced yes)
-		(property "Reference" "#PWR029"
+		(property "Reference" "#PWR046"
 			(at 449.58 123.19 0)
 			(hide yes)
@@
 			(project "PDB"
 				(path "/a9cf05c4-aac5-4cf1-b700-1d3045f8dfbd/a24fc02a-90d5-41f1-96d5-cd0fa3bff83a"
-					(reference "#PWR029")
+					(reference "#PWR046")
 					(unit 1)
 				)
@@
 			)
 		)
-		(property "Footprint" "Resistor_SMD:R_0603_1608Metric"
+		(property "Footprint" "Resistor_SMD:R_Shunt_Vishay_WSR2_WSR3_KelvinConnection"
 			(at 439.42 124.968 90)
 			(hide yes)
@@
 		(dnp no)
 		(fields_autoplaced yes)
-		(property "Reference" "#PWR052"
+		(property "Reference" "#PWR042"
 			(at 419.1 120.65 0)
 			(hide yes)
@@
 			(project "PDB"
 				(path "/a9cf05c4-aac5-4cf1-b700-1d3045f8dfbd/a24fc02a-90d5-41f1-96d5-cd0fa3bff83a"
-					(reference "#PWR052")
+					(reference "#PWR042")
 					(unit 1)
 				)
@@
 		(dnp no)
 		(fields_autoplaced yes)
-		(property "Reference" "#PWR027"
+		(property "Reference" "#PWR040"
 			(at 359.41 147.32 0)
 			(hide yes)
@@
 			(project "PDB"
 				(path "/a9cf05c4-aac5-4cf1-b700-1d3045f8dfbd/a24fc02a-90d5-41f1-96d5-cd0fa3bff83a"
-					(reference "#PWR027")
+					(reference "#PWR040")
 					(unit 1)
 				)
@@
 		(dnp no)
 		(fields_autoplaced yes)
-		(property "Reference" "#PWR069"
+		(property "Reference" "#PWR047"
 			(at 476.25 135.89 0)
 			(hide yes)
@@
 			(project "PDB"
 				(path "/a9cf05c4-aac5-4cf1-b700-1d3045f8dfbd/a24fc02a-90d5-41f1-96d5-cd0fa3bff83a"
-					(reference "#PWR069")
+					(reference "#PWR047")
 					(unit 1)
 				)
@@
 		(dnp no)
 		(fields_autoplaced yes)
-		(property "Reference" "#PWR053"
+		(property "Reference" "#PWR045"
 			(at 459.74 104.14 0)
 			(hide yes)
@@
 			(project "PDB"
 				(path "/a9cf05c4-aac5-4cf1-b700-1d3045f8dfbd/a24fc02a-90d5-41f1-96d5-cd0fa3bff83a"
-					(reference "#PWR053")
+					(reference "#PWR045")
 					(unit 1)
 				)
@@
 		(dnp no)
 		(fields_autoplaced yes)
-		(property "Reference" "#PWR028"
+		(property "Reference" "#PWR037"
 			(at 149.86 95.25 0)
 			(hide yes)
@@
 			(project "PDB"
 				(path "/a9cf05c4-aac5-4cf1-b700-1d3045f8dfbd/a24fc02a-90d5-41f1-96d5-cd0fa3bff83a"
-					(reference "#PWR028")
+					(reference "#PWR037")
 					(unit 1)
 				)
@@
 		(dnp no)
 		(fields_autoplaced yes)
-		(property "Reference" "#PWR023"
+		(property "Reference" "#PWR043"
 			(at 427.99 203.2 0)
 			(hide yes)
@@
 			(project "PDB"
 				(path "/a9cf05c4-aac5-4cf1-b700-1d3045f8dfbd/a24fc02a-90d5-41f1-96d5-cd0fa3bff83a"
-					(reference "#PWR023")
+					(reference "#PWR043")
 					(unit 1)
 				)
@@
 		(dnp no)
 		(fields_autoplaced yes)
-		(property "Reference" "#PWR026"
+		(property "Reference" "#PWR038"
 			(at 222.25 209.55 0)
 			(hide yes)
@@
 			(project "PDB"
 				(path "/a9cf05c4-aac5-4cf1-b700-1d3045f8dfbd/a24fc02a-90d5-41f1-96d5-cd0fa3bff83a"
-					(reference "#PWR026")
+					(reference "#PWR038")
 					(unit 1)
 				)

Commit message: lots of routing
Parts:
- R21: footprint Resistor_SMD:R_Shunt_Vishay_WSR2_WSR3_KelvinConnection -> Resistor_SMD:R_Shunt_Vishay_WSK2512_6332Metric_T2.66mm
Changed lines of the file:
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@@
 			)
 		)
-		(property "Footprint" "Resistor_SMD:R_Shunt_Vishay_WSR2_WSR3_KelvinConnection"
+		(property "Footprint" "Resistor_SMD:R_Shunt_Vishay_WSK2512_6332Metric_T2.66mm"
 			(at 439.42 124.968 90)
 			(hide yes)
