File: PDB/5v_4a.kicad_sch (KiCad schematic)
At the start: 18 parts, among them U10 LM76005RNPR, U11 INA228

Commit message: laid out many, many things
Parts:
- R24: footprint Resistor_SMD:R_Shunt_Vishay_WSR2_WSR3_KelvinConnection -> Resistor_SMD:R_Shunt_Vishay_WSK2512_6332Metric_T2.66mm
Changed lines of the file:
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@@
 			)
 		)
-		(property "Footprint" "Resistor_SMD:R_Shunt_Vishay_WSR2_WSR3_KelvinConnection"
+		(property "Footprint" "Resistor_SMD:R_Shunt_Vishay_WSK2512_6332Metric_T2.66mm"
 			(at 188.722 90.17 90)
 			(hide yes)

Commit message: coordinated labels in schem
Labeled all components to be Rxx, Cxx, ext forms through all sheets so labels for BOM and layout are work together as one long list.
Parts:
- renumbered Cin2 to C26, Cinx2 to C27, Cvcc2 to C28, Cboot2 to C29, Cout2 to C30, Coutx1 to C31, C16 to C32, Rpgood1 to R27, Rfbt2 to R28, Rfbb2 to R29, R23 to R30, R24 to R31
Changed lines of the file:
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@@
 		(dnp no)
 		(fields_autoplaced yes)
-		(property "Reference" "R24"
+		(property "Reference" "R31"
 			(at 187.96 88.8999 0)
 			(show_name no)
@@
 			(project "PDB"
 				(path "/a9cf05c4-aac5-4cf1-b700-1d3045f8dfbd/fb4943bd-b408-4249-996b-df676f2bb727"
-					(reference "R24")
+					(reference "R31")
 					(unit 1)
 				)
@@
 		(dnp no)
 		(fields_autoplaced yes)
-		(property "Reference" "#PWR054"
+		(property "Reference" "#PWR055"
 			(at 193.04 69.85 0)
 			(hide yes)
@@
 			(project "PDB"
 				(path "/a9cf05c4-aac5-4cf1-b700-1d3045f8dfbd/fb4943bd-b408-4249-996b-df676f2bb727"
-					(reference "#PWR054")
+					(reference "#PWR055")
 					(unit 1)
 				)
@@
 		(dnp no)
 		(fields_autoplaced yes)
-		(property "Reference" "Cinx2"
+		(property "Reference" "C27"
 			(at 52.07 88.8999 0)
 			(show_name no)
@@
 			(project "PDB"
 				(path "/a9cf05c4-aac5-4cf1-b700-1d3045f8dfbd/fb4943bd-b408-4249-996b-df676f2bb727"
-					(reference "Cinx2")
+					(reference "C27")
 					(unit 1)
 				)
@@
 		(dnp no)
 		(fields_autoplaced yes)
-		(property "Reference" "#PWR050"
+		(property "Reference" "#PWR051"
 			(at 100.33 120.65 0)
 			(hide yes)
@@
 			(project "PDB"
 				(path "/a9cf05c4-aac5-4cf1-b700-1d3045f8dfbd/fb4943bd-b408-4249-996b-df676f2bb727"
-					(reference "#PWR050")
+					(reference "#PWR051")
 					(unit 1)
 				)
@@
 		(dnp no)
 		(fields_autoplaced yes)
-		(property "Reference" "Rfbt2"
+		(property "Reference" "R28"
 			(at 140.97 82.5499 0)
 			(show_name no)
@@
 			(project "PDB"
 				(path "/a9cf05c4-aac5-4cf1-b700-1d3045f8dfbd/fb4943bd-b408-4249-996b-df676f2bb727"
-					(reference "Rfbt2")
+					(reference "R28")
 					(unit 1)
 				)
@@
 		(dnp no)
 		(fields_autoplaced yes)
-		(property "Reference" "Coutx1"
+		(property "Reference" "C31"
 			(at 172.72 91.4399 0)
 			(show_name no)
@@
 			(project "PDB"
 				(path "/a9cf05c4-aac5-4cf1-b700-1d3045f8dfbd/fb4943bd-b408-4249-996b-df676f2bb727"
-					(reference "Coutx1")
+					(reference "C31")
 					(unit 1)
 				)
@@
 		(dnp no)
 		(fields_autoplaced yes)
-		(property "Reference" "#PWR056"
+		(property "Reference" "#PWR057"
 			(at 228.6 81.28 0)
 			(hide yes)
@@
 			(project "PDB"
 				(path "/a9cf05c4-aac5-4cf1-b700-1d3045f8dfbd/fb4943bd-b408-4249-996b-df676f2bb727"
-					(reference "#PWR056")
+					(reference "#PWR057")
 					(unit 1)
 				)
@@
 		(dnp no)
 		(fields_autoplaced yes)
-		(property "Reference" "Rpgood1"
+		(property "Reference" "R27"
 			(at 125.73 82.5499 0)
 			(show_name no)
@@
 			(project "PDB"
 				(path "/a9cf05c4-aac5-4cf1-b700-1d3045f8dfbd/fb4943bd-b408-4249-996b-df676f2bb727"
-					(reference "Rpgood1")
+					(reference "R27")
 					(unit 1)
 				)
@@
 		(dnp no)
 		(fields_autoplaced yes)
-		(property "Reference" "Rfbb2"
+		(property "Reference" "R29"
 			(at 140.97 97.7899 0)
 			(show_name no)
@@
 			(project "PDB"
 				(path "/a9cf05c4-aac5-4cf1-b700-1d3045f8dfbd/fb4943bd-b408-4249-996b-df676f2bb727"
-					(reference "Rfbb2")
+					(reference "R29")
 					(unit 1)
 				)
@@
 		(dnp no)
 		(fields_autoplaced yes)
-		(property "Reference" "C16"
+		(property "Reference" "C32"
 			(at 205.74 62.23 90)
 			(show_name no)
@@
 			(project "PDB"
 				(path "/a9cf05c4-aac5-4cf1-b700-1d3045f8dfbd/fb4943bd-b408-4249-996b-df676f2bb727"
-					(reference "C16")
+					(reference "C32")
 					(unit 1)
 				)
@@
 		(dnp no)
 		(fields_autoplaced yes)
-		(property "Reference" "#PWR051"
+		(property "Reference" "#PWR052"
 			(at 101.6 78.74 0)
 			(hide yes)
@@
 			(project "PDB"
 				(path "/a9cf05c4-aac5-4cf1-b700-1d3045f8dfbd/fb4943bd-b408-4249-996b-df676f2bb727"
-					(reference "#PWR051")
+					(reference "#PWR052")
 					(unit 1)
 				)
@@
 		(dnp no)
 		(fields_autoplaced yes)
-		(property "Reference" "Cvcc2"
+		(property "Reference" "C28"
 			(at 105.41 64.7699 0)
 			(show_name no)
@@
 			(project "PDB"
 				(path "/a9cf05c4-aac5-4cf1-b700-1d3045f8dfbd/fb4943bd-b408-4249-996b-df676f2bb727"
-					(reference "Cvcc2")
+					(reference "C28")
 					(unit 1)
 				)
@@
 		(dnp no)
 		(fields_autoplaced yes)
-		(property "Reference" "#PWR049"
+		(property "Reference" "#PWR050"
 			(at 99.06 95.25 0)
 			(hide yes)
@@
 			(project "PDB"
 				(path "/a9cf05c4-aac5-4cf1-b700-1d3045f8dfbd/fb4943bd-b408-4249-996b-df676f2bb727"
-					(reference "#PWR049")
+					(reference "#PWR050")
 					(unit 1)
 				)
@@
 		(dnp no)
 		(fields_autoplaced yes)
-		(property "Reference" "#PWR052"
+		(property "Reference" "#PWR053"
 			(at 176.53 128.27 0)
 			(hide yes)
@@
 			(project "PDB"
 				(path "/a9cf05c4-aac5-4cf1-b700-1d3045f8dfbd/fb4943bd-b408-4249-996b-df676f2bb727"
-					(reference "#PWR052")
+					(reference "#PWR053")
 					(unit 1)
 				)
@@
 		(dnp no)
 		(fields_autoplaced yes)
-		(property "Reference" "Cout2"
+		(property "Reference" "C30"
 			(at 160.02 91.6939 0)
 			(show_name no)
@@
 			(project "PDB"
 				(path "/a9cf05c4-aac5-4cf1-b700-1d3045f8dfbd/fb4943bd-b408-4249-996b-df676f2bb727"
-					(reference "Cout2")
+					(reference "C30")
 					(unit 1)
 				)
@@
 		(dnp no)
 		(fields_autoplaced yes)
-		(property "Reference" "Cboot2"
+		(property "Reference" "C29"
 			(at 113.03 81.2799 0)
 			(show_name no)
@@
 			(project "PDB"
 				(path "/a9cf05c4-aac5-4cf1-b700-1d3045f8dfbd/fb4943bd-b408-4249-996b-df676f2bb727"
-					(reference "Cboot2")
+					(reference "C29")
 					(unit 1)
 				)
@@
 		(dnp no)
 		(fields_autoplaced yes)
-		(property "Reference" "#PWR055"
+		(property "Reference" "#PWR056"
 			(at 209.55 110.49 0)
 			(hide yes)
@@
 			(project "PDB"
 				(path "/a9cf05c4-aac5-4cf1-b700-1d3045f8dfbd/fb4943bd-b408-4249-996b-df676f2bb727"
-					(reference "#PWR055")
+					(reference "#PWR056")
 					(unit 1)
 				)
@@
 		(dnp no)
 		(fields_autoplaced yes)
-		(property "Reference" "Cin2"
+		(property "Reference" "C26"
 			(at 40.64 88.8999 0)
 			(show_name no)
@@
 			(project "PDB"
 				(path "/a9cf05c4-aac5-4cf1-b700-1d3045f8dfbd/fb4943bd-b408-4249-996b-df676f2bb727"
-					(reference "Cin2")
+					(reference "C26")
 					(unit 1)
 				)
@@
 		(dnp no)
 		(fields_autoplaced yes)
-		(property "Reference" "#PWR048"
+		(property "Reference" "#PWR049"
 			(at 36.83 82.55 0)
 			(hide yes)
@@
 			(project "PDB"
 				(path "/a9cf05c4-aac5-4cf1-b700-1d3045f8dfbd/fb4943bd-b408-4249-996b-df676f2bb727"
-					(reference "#PWR048")
+					(reference "#PWR049")
 					(unit 1)
 				)
@@
 		(dnp no)
 		(fields_autoplaced yes)
-		(property "Reference" "#PWR053"
+		(property "Reference" "#PWR054"
 			(at 190.5 100.33 0)
 			(hide yes)
@@
 			(project "PDB"
 				(path "/a9cf05c4-aac5-4cf1-b700-1d3045f8dfbd/fb4943bd-b408-4249-996b-df676f2bb727"
-					(reference "#PWR053")
+					(reference "#PWR054")
 					(unit 1)
 				)
@@
 		(in_pos_files yes)
 		(dnp no)
-		(property "Reference" "R23"
+		(property "Reference" "R30"
 			(at 179.07 104.1399 0)
 			(show_name no)
@@
 			(project "PDB"
 				(path "/a9cf05c4-aac5-4cf1-b700-1d3045f8dfbd/fb4943bd-b408-4249-996b-df676f2bb727"
-					(reference "R23")
-					(unit 1)
-				)
+					(reference "R30")
+					(unit 1)
+				)

Commit message: last push before removing oring
i think we're going with an interlock system instead. the battery oring on here will take far too much physical room on the board to make it worthwhile. this push removes the oring and assumes a single power input.
Parts:
- U10: footprint Dependencies:LM76005RNPR -> LM76005RNPR:QFN50P600X400X80-31N
Connections:
- net at R31.2: no longer U11.10 (Vin+)
- net at R31.3: no longer U11.9 (Vin-)
Changed lines of the file:
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@@
 			)
 		)
-		(property "Footprint" "Dependencies:LM76005RNPR"
+		(property "Footprint" "LM76005RNPR:QFN50P600X400X80-31N"
 			(at 78.74 91.44 0)
 			(hide yes)
