File: PDB/USBCPD.kicad_sch (KiCad schematic)
At the start: 50 parts, among them J1 USB_C_Receptacle, Q3 STL6P3LLH6, Q4 STL6P3LLH6, U19 INA228, U6 ST1S14PHR, U7 STUSB4700YQTR, U8 STR2P3LLH6, U9 LM76005QRNPRQ1

Commit message: Finished all the footprints. doing poe myself now
finally.
Parts:
- C38: renamed from C36; footprint Capacitor_SMD:C_1206_3216Metric -> Capacitor_SMD:C_0603_1608Metric
- D19: renamed from D8; footprint (none) -> Package_TO_SOT_SMD:TO-252-2
- F5: renamed from F4; footprint (none) -> Fuse:Fuse_1206_3216Metric
- J14: renamed from J1; footprint (none) -> Connector_USB:USB_C_Receptacle_CNCTech_C-ARA1-AK51X
- L5: renamed from L2; footprint (none) -> Inductor_SMD:L_1206_3216Metric
- L6: renamed from L3; footprint (none) -> Inductor_SMD:L_1206_3216Metric
- R43: renamed from R41; footprint (none) -> Resistor_SMD:R_0603_1608Metric
- U16: renamed from U9; footprint RNP0030A -> Dependencies:RNP0030A
- U17: renamed from U6; footprint HSOP8_STM -> Dependencies:HSOP8_STM
- U18: renamed from U7; footprint QFN_700QTR_STM -> Dependencies:QFN_700QTR_STM
- U19: renamed from U8; footprint SOT_3LLH6_STM -> Dependencies:SOT_3LLH6_STM
- U20: renamed from U19; footprint Package_SO:TSSOP-10_3x3mm_P0.5mm -> Package_SO:HVSSOP-10-1EP_3x3mm_P0.5mm_EP1.83x1.89mm
- renumbered C1 to C20, C2 to C21, C12 to C22, C3 to C23, C4 to C24, C5 to C25, C6 to C26, C7 to C27, C14 to C28, C15 to C29, C16 to C30, C18 to C31, C22 to C32, C23 to C33, C24 to C34, C27 to C35, C26 to C36, C25 to C37, C28 to C39, D19 to D20, Q3 to Q7, Q4 to Q8, R1 to R29, R2 to R30, R3 to R31, R4 to R32, R5 to R33, R7 to R34, R10 to R35, R11 to R36, R12 to R37, R13 to R38, R15 to R39, R14 to R40, R17 to R41, R18 to R42, R46 to R44

Commit message: more footprint
Parts:
- Q7, Q8: footprint STL6P3LLH6:TRANS_STL6P3LLH6 -> Dependencies:CSD19502Q5B
- U16: footprint Dependencies:RNP0030A -> Dependencies:LM76005RNPR
Changed lines of the file:
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@@
 			)
 		)
-		(property "Footprint" "STL6P3LLH6:TRANS_STL6P3LLH6"
+		(property "Footprint" "Dependencies:CSD19502Q5B"
 			(at 416.56 157.48 0)
 			(hide yes)
@@
 			)
 		)
-		(property "Footprint" "STL6P3LLH6:TRANS_STL6P3LLH6"
+		(property "Footprint" "Dependencies:CSD19502Q5B"
 			(at 438.15 162.56 0)
 			(hide yes)
@@
 			)
 		)
-		(property "Footprint" "Dependencies:RNP0030A"
+		(property "Footprint" "Dependencies:LM76005RNPR"
 			(at 107.95 180.34 0)
 			(hide yes)

Commit message: fixed component footprints
Parts:
- R43: footprint Resistor_SMD:R_0603_1608Metric -> Resistor_SMD:R_Shunt_Vishay_WSR2_WSR3_KelvinConnection
Changed lines of the file:
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@@
 		(dnp no)
 		(fields_autoplaced yes)
-		(property "Reference" "#PWR037"
+		(property "Reference" "#PWR084"
 			(at 359.41 179.07 0)
 			(hide yes)
@@
 			(project "PDB"
 				(path "/a9cf05c4-aac5-4cf1-b700-1d3045f8dfbd/b0911c37-41be-485e-baed-d6c7fecee207"
-					(reference "#PWR037")
+					(reference "#PWR084")
 					(unit 1)
 				)
@@
 		(dnp no)
 		(fields_autoplaced yes)
-		(property "Reference" "#PWR073"
+		(property "Reference" "#PWR090"
 			(at 514.35 152.4 0)
 			(hide yes)
@@
 			(project "PDB"
 				(path "/a9cf05c4-aac5-4cf1-b700-1d3045f8dfbd/b0911c37-41be-485e-baed-d6c7fecee207"
-					(reference "#PWR073")
+					(reference "#PWR090")
 					(unit 1)
 				)
@@
 		(dnp no)
 		(fields_autoplaced yes)
-		(property "Reference" "#PWR033"
+		(property "Reference" "#PWR080"
 			(at 317.5 180.34 0)
 			(hide yes)
@@
 			(project "PDB"
 				(path "/a9cf05c4-aac5-4cf1-b700-1d3045f8dfbd/b0911c37-41be-485e-baed-d6c7fecee207"
-					(reference "#PWR033")
+					(reference "#PWR080")
 					(unit 1)
 				)
@@
 		(dnp no)
 		(fields_autoplaced yes)
-		(property "Reference" "#PWR065"
+		(property "Reference" "#PWR089"
 			(at 499.11 127 0)
 			(hide yes)
@@
 			(project "PDB"
 				(path "/a9cf05c4-aac5-4cf1-b700-1d3045f8dfbd/b0911c37-41be-485e-baed-d6c7fecee207"
-					(reference "#PWR065")
+					(reference "#PWR089")
 					(unit 1)
 				)
@@
 		(dnp no)
 		(fields_autoplaced yes)
-		(property "Reference" "#PWR035"
+		(property "Reference" "#PWR083"
 			(at 340.36 185.42 0)
 			(hide yes)
@@
 			(project "PDB"
 				(path "/a9cf05c4-aac5-4cf1-b700-1d3045f8dfbd/b0911c37-41be-485e-baed-d6c7fecee207"
-					(reference "#PWR035")
+					(reference "#PWR083")
 					(unit 1)
 				)
@@
 		(dnp no)
 		(fields_autoplaced yes)
-		(property "Reference" "#PWR066"
+		(property "Reference" "#PWR087"
 			(at 467.36 102.87 0)
 			(hide yes)
@@
 			(project "PDB"
 				(path "/a9cf05c4-aac5-4cf1-b700-1d3045f8dfbd/b0911c37-41be-485e-baed-d6c7fecee207"
-					(reference "#PWR066")
+					(reference "#PWR087")
 					(unit 1)
 				)
@@
 		(dnp no)
 		(fields_autoplaced yes)
-		(property "Reference" "#PWR039"
+		(property "Reference" "#PWR088"
 			(at 467.36 176.53 0)
 			(hide yes)
@@
 			(project "PDB"
 				(path "/a9cf05c4-aac5-4cf1-b700-1d3045f8dfbd/b0911c37-41be-485e-baed-d6c7fecee207"
-					(reference "#PWR039")
+					(reference "#PWR088")
 					(unit 1)
 				)
@@
 		(dnp no)
 		(fields_autoplaced yes)
-		(property "Reference" "#PWR038"
+		(property "Reference" "#PWR085"
 			(at 393.7 186.69 0)
 			(hide yes)
@@
 			(project "PDB"
 				(path "/a9cf05c4-aac5-4cf1-b700-1d3045f8dfbd/b0911c37-41be-485e-baed-d6c7fecee207"
-					(reference "#PWR038")
+					(reference "#PWR085")
 					(unit 1)
 				)
@@
 		(dnp no)
 		(fields_autoplaced yes)
-		(property "Reference" "#PWR036"
+		(property "Reference" "#PWR081"
 			(at 326.39 243.84 0)
 			(hide yes)
@@
 			(project "PDB"
 				(path "/a9cf05c4-aac5-4cf1-b700-1d3045f8dfbd/b0911c37-41be-485e-baed-d6c7fecee207"
-					(reference "#PWR036")
+					(reference "#PWR081")
 					(unit 1)
 				)
@@
 		(dnp no)
 		(fields_autoplaced yes)
-		(property "Reference" "#PWR030"
+		(property "Reference" "#PWR075"
 			(at 52.07 158.75 0)
 			(hide yes)
@@
 			(project "PDB"
 				(path "/a9cf05c4-aac5-4cf1-b700-1d3045f8dfbd/b0911c37-41be-485e-baed-d6c7fecee207"
-					(reference "#PWR030")
+					(reference "#PWR075")
 					(unit 1)
 				)
@@
 		(dnp no)
 		(fields_autoplaced yes)
-		(property "Reference" "#PWR031"
+		(property "Reference" "#PWR077"
 			(at 81.28 153.67 0)
 			(hide yes)
@@
 			(project "PDB"
 				(path "/a9cf05c4-aac5-4cf1-b700-1d3045f8dfbd/b0911c37-41be-485e-baed-d6c7fecee207"
-					(reference "#PWR031")
+					(reference "#PWR077")
 					(unit 1)
 				)
@@
 		(dnp no)
 		(fields_autoplaced yes)
-		(property "Reference" "#PWR04"
+		(property "Reference" "#PWR076"
 			(at 68.58 223.52 0)
 			(hide yes)
@@
 			(project "PDB"
 				(path "/a9cf05c4-aac5-4cf1-b700-1d3045f8dfbd/b0911c37-41be-485e-baed-d6c7fecee207"
-					(reference "#PWR04")
+					(reference "#PWR076")
 					(unit 1)
 				)
@@
 		(dnp no)
 		(fields_autoplaced yes)
-		(property "Reference" "#PWR034"
+		(property "Reference" "#PWR082"
 			(at 330.2 180.34 0)
 			(hide yes)
@@
 			(project "PDB"
 				(path "/a9cf05c4-aac5-4cf1-b700-1d3045f8dfbd/b0911c37-41be-485e-baed-d6c7fecee207"
-					(reference "#PWR034")
+					(reference "#PWR082")
 					(unit 1)
 				)
@@
 			)
 		)
-		(property "Footprint" "Resistor_SMD:R_0603_1608Metric"
+		(property "Footprint" "Resistor_SMD:R_Shunt_Vishay_WSR2_WSR3_KelvinConnection"
 			(at 478.79 147.828 90)
 			(hide yes)
@@
 		(dnp no)
 		(fields_autoplaced yes)
-		(property "Reference" "#PWR064"
+		(property "Reference" "#PWR086"
 			(at 458.47 143.51 0)
 			(hide yes)
@@
 			(project "PDB"
 				(path "/a9cf05c4-aac5-4cf1-b700-1d3045f8dfbd/b0911c37-41be-485e-baed-d6c7fecee207"
-					(reference "#PWR064")
+					(reference "#PWR086")
 					(unit 1)
 				)
@@
 		(dnp no)
 		(fields_autoplaced yes)
-		(property "Reference" "#PWR040"
+		(property "Reference" "#PWR091"
 			(at 523.24 147.32 0)
 			(hide yes)
@@
 			(project "PDB"
 				(path "/a9cf05c4-aac5-4cf1-b700-1d3045f8dfbd/b0911c37-41be-485e-baed-d6c7fecee207"
-					(reference "#PWR040")
+					(reference "#PWR091")
 					(unit 1)
 				)
@@
 		(dnp no)
 		(fields_autoplaced yes)
-		(property "Reference" "#PWR032"
+		(property "Reference" "#PWR079"
 			(at 217.17 200.66 0)
 			(hide yes)
@@
 			(project "PDB"
 				(path "/a9cf05c4-aac5-4cf1-b700-1d3045f8dfbd/b0911c37-41be-485e-baed-d6c7fecee207"
-					(reference "#PWR032")
+					(reference "#PWR079")
 					(unit 1)
 				)
@@
 		(dnp no)
 		(fields_autoplaced yes)
-		(property "Reference" "#PWR07"
+		(property "Reference" "#PWR078"
 			(at 129.54 181.1381 0)
 			(hide yes)
@@
 			(project "PDB"
 				(path "/a9cf05c4-aac5-4cf1-b700-1d3045f8dfbd/b0911c37-41be-485e-baed-d6c7fecee207"
-					(reference "#PWR07")
+					(reference "#PWR078")
 					(unit 1)
 				)

Commit message: lots of routing
Parts:
- R43: footprint Resistor_SMD:R_Shunt_Vishay_WSR2_WSR3_KelvinConnection -> Resistor_SMD:R_Shunt_Vishay_WSK2512_6332Metric_T2.66mm
Changed lines of the file:
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@@
 	(wire
 		(pts
-			(xy 118.11 160.02) (xy 125.73 160.02)
-		)
-		(stroke
-			(width 0)
-			(type default)
-		)
-	)
-	(wire
-		(pts
 			(xy 452.12 160.02) (xy 452.12 198.12)
 		)
@@
 			)
 		)
-		(property "Footprint" "Resistor_SMD:R_Shunt_Vishay_WSR2_WSR3_KelvinConnection"
+		(property "Footprint" "Resistor_SMD:R_Shunt_Vishay_WSK2512_6332Metric_T2.66mm"
 			(at 478.79 147.828 90)
 			(hide yes)

Commit message: coordinated labels in schem
Labeled all components to be Rxx, Cxx, ext forms through all sheets so labels for BOM and layout are work together as one long list.
Parts:
- renumbered C20 to C48, C21 to C49, C22 to C50, C23 to C51, C24 to C52, C25 to C53, C26 to C54, C27 to C55, C28 to C56, C29 to C57, C30 to C58, C31 to C59, C32 to C60, C33 to C61, C34 to C62, C35 to C63, C36 to C64, C37 to C65, C38 to C66, C39 to C67, J14 to J13, Q8 to Q10, Q7 to Q9, R29 to R47, R30 to R48, R31 to R49, R32 to R50, R33 to R51, R34 to R52, R35 to R53, R36 to R54, R37 to R55, R38 to R56, R39 to R57, R40 to R58, R41 to R59, R42 to R60, R43 to R61, R44 to R62

Commit message: init comit for eth demo
Parts:
- Q10, Q9: footprint Dependencies:CSD19502Q5B -> STL6P3LLH6:TRANS_STL6P3LLH6
Connections:
- net at R59.1, R60.2: now also Q10.G1 (G), Q9.G1 (G); no longer Q10.4, Q9.4
- net at C60.1, C61.1, C62.1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: now also Q9.D1 (D); no longer Q9.5_8
- net at F5.1, U18.18 (VBUS_SENSE): now also Q10.D1 (D); no longer Q10.5_8
- new net: Q10.S1 (S), Q9.S1 (S), R59.2
Changed lines of the file:
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@@
 	)
 	(symbol
+		(lib_name "STL6P3LLH6_1")
 		(lib_id "sym&foot:STL6P3LLH6")
 		(at 416.56 157.48 270)
@@
 			)
 		)
-		(property "Footprint" "Dependencies:CSD19502Q5B"
+		(property "Footprint" "STL6P3LLH6:TRANS_STL6P3LLH6"
 			(at 416.56 157.48 0)
 			(hide yes)
@@
 			)
 		)
-		(pin "4"
-		)
-		(pin "2"
-		)
-		(pin "1"
-		)
-		(pin "5_8"
-		)
-		(pin "3"
+		(pin "D1"
+		)
+		(pin "G1"
+		)
+		(pin "S1"
 		)
 		(instances
@@
 			)
 		)
-		(property "Footprint" "Dependencies:CSD19502Q5B"
+		(property "Footprint" "STL6P3LLH6:TRANS_STL6P3LLH6"
 			(at 438.15 162.56 0)
 			(hide yes)
@@
 			)
 		)
-		(pin "4"
-		)
-		(pin "2"
-		)
-		(pin "1"
-		)
-		(pin "5_8"
-		)
-		(pin "3"
-		)
-		(instances
+		(pin "G1"
+		)
+		(pin "D1"
+		)
+		(pin "S1"
+		)
+		(instances

Commit message: last push before removing oring
i think we're going with an interlock system instead. the battery oring on here will take far too much physical room on the board to make it worthwhile. this push removes the oring and assumes a single power input.
Parts:
- U16: footprint Dependencies:LM76005RNPR -> RNP0030A
- U17: footprint Dependencies:HSOP8_STM -> HSOP8_STM
- U18: footprint Dependencies:QFN_700QTR_STM -> QFN_700QTR_STM
- U19: footprint Dependencies:SOT_3LLH6_STM -> SOT_3LLH6_STM
- U20: footprint Package_SO:HVSSOP-10-1EP_3x3mm_P0.5mm_EP1.83x1.89mm -> Package_SO:TSSOP-10_3x3mm_P0.5mm
Connections:
- net +10VDC: no longer U17.5 (EN2), U17.7 (VIN)
- net GND: now also U18.12 (GPIO0); no longer U17.3 (*EN1), U17.6 (GND), U17.EPAD, U18.10 (GND), U18.22 (VSYS), U18.25 (EP), U18.3 (VCONN), U18.6 (RESET)
- net SCL: now also U18.9 (ALERT-); no longer U18.7 (SCL)
- net SDA: no longer U18.8 (SDA)
- net at C64.2: no longer U18.21 (VREG_1V2)
- net at R52.1, R53.2: now also U18.3 (VCONN); no longer U18.14 (GPIO2)
- net at R51.1, R52.2: no longer U18.15 (GPIO3)
- net at R60.1: now also U18.24 (VDD); no longer U18.20 (VBUS_EN_SRC)
- net at C60.1, C61.1, C62.1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: no longer U18.24 (VDD)
- net at R54.1, R55.2: now also U18.6 (RESET); no longer U18.12 (GPIO0)
- net at R53.1, R54.2: no longer U18.11 (GPIO1)
- net at C59.2: no longer U17.1 (BOOT)
- net at C60.2, R50.1, R51.2: no longer U17.4 (FB)
- net at U17.8 (SW): no longer L6.1
- net at U18.13 (VVAR_ADDR0): no longer R56.2
- net at F5.1, Q10.D1 (D): no longer U18.18 (VBUS_SENSE)
- net at R58.1, U19.1 (G): no longer U18.19 (VBUS_DISCH)
- net at J13.A5 (CC1): now also U18.14 (GPIO2); no longer U18.2 (CC1)
- net at U18.23 (VREG_2V7): no longer C65.2
- net at U18.4 (CC2): no longer J13.B5 (CC2)
- net at R61.4, R62.1, TP10.1: no longer J13.A4 (VBUS)
- net at J13.A9 (VBUS), J13.B4 (VBUS), J13.B9 (VBUS): now also J13.A4 (VBUS)
- net at R61.2: no longer U20.10 (Vin+)
- net at R61.3: no longer U20.9 (Vin-)
Changed lines of the file:
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@@
 	)
 	(symbol
-		(lib_name "STL6P3LLH6_1")
 		(lib_id "sym&foot:STL6P3LLH6")
 		(at 416.56 157.48 270)
@@
 			)
 		)
-		(property "Footprint" "Dependencies:HSOP8_STM"
+		(property "Footprint" "HSOP8_STM"
 			(at 233.68 161.29 0)
 			(hide yes)
@@
 			)
 		)
-		(property "Footprint" "Dependencies:QFN_700QTR_STM"
+		(property "Footprint" "QFN_700QTR_STM"
 			(at 307.848 170.18 0)
 			(hide yes)
@@
 			)
 		)
-		(property "Footprint" "Package_SO:HVSSOP-10-1EP_3x3mm_P0.5mm_EP1.83x1.89mm"
+		(property "Footprint" "Package_SO:TSSOP-10_3x3mm_P0.5mm"
 			(at 452.374 102.108 0)
 			(hide yes)
@@
 			)
 		)
-		(property "Footprint" "Dependencies:SOT_3LLH6_STM"
+		(property "Footprint" "SOT_3LLH6_STM"
 			(at 389.89 168.91 0)
 			(hide yes)
@@
 			)
 		)
-		(property "Footprint" "Dependencies:LM76005RNPR"
+		(property "Footprint" "RNP0030A"
 			(at 107.95 180.34 0)
 			(hide yes)
