File: PDB/PDB.kicad_pcb (KiCad board)
At the start: 2 copper layers, 130 x 112.6 mm, 259 parts, among them J1 Micro_SD_Card, J10 XT90PW-M, J11 XT90PW-M, J12 XT90PW-M, J14 USB_C_Receptacle, J15 RJ45_Abracon_ARJP11A-MASA-B-A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, J2 UART OUT, J3 swd, J4 XT30PW-M, J5 XT30PW-M, J6 XT60PW-M, J7 XT90PW-M, J8 XT90PW-M, J9 XT90PW-M, M1 GENERIC_MOSFET_N, M2 GENERIC_MOSFET_N, M3 CSD19502Q5B, M4 CSD17578Q3A, Q1 IPT012N08N5, Q2 IPT012N08N5, Q3 BSC093N15NS5, Q4 BSC093N15NS5, Q5 CSD19502Q5B, Q7 STL6P3LLH6, Q8 STL6P3LLH6, U1 STM32H742VGTx, U10 LM76005RNPR, U11 INA228, U12 TLV62569ADRLR, U13 INA228, U14 LM5118MH, U15 INA228, U16 LM76005QRNPRQ1, U17 ST1S14PHR, U18 STUSB4700YQTR, U19 STR2P3LLH6, U2 MCP9804_DFN, U20 INA228, U21 LM5118MH/NOPB, U22 INA228, U3 MCP9804_DFN, U4 MCP9804_DFN, U5 LTC4359-DCB, U6 LTC4359-DCB, U7 TMCS1108A4UQDRQ1, U8 LM5116MH/NOPB, U9 INA228

Commit message: laid out many, many things
Parts:
- added Q6: CSD19537Q3, Dependencies:CSD19537Q3, F.Cu at (415.9, 189.3)
- R24, R26, R27: footprint Resistor_SMD:R_Shunt_Vishay_WSR2_WSR3_KelvinConnection -> Resistor_SMD:R_Shunt_Vishay_WSK2512_6332Metric_T2.66mm
- moved C17 161.8 mm to (539.1, 178.0)
- moved Cout3 153.0 mm to (533.6, 174.2), turned to 180 degrees
- moved U13 152.6 mm to (537.2, 182.0), turned to 90 degrees
- moved R25 152.5 mm to (530.3, 182.4), turned to 90 degrees
- moved Cin3 150.7 mm to (530.2, 173.5)
- moved R26 147.4 mm to (533.1, 179.5), turned to -90 degrees
- moved TP8 147.2 mm to (529.9, 185.8), turned to 90 degrees
- moved Rfbb3 145.6 mm to (530.2, 168.0)
- moved Rfbt3 145.3 mm to (530.2, 169.7), turned to 180 degrees
- moved F3 142.1 mm to (536.3, 175.7), turned to 90 degrees
- moved L3 140.1 mm to (534.4, 172.0)
- moved U12 138.5 mm to (530.1, 171.5)
- moved D15 136.6 mm to (529.3, 179.8)
- moved C19 131.1 mm to (418.4, 199.0), turned to 90 degrees
- moved Cout4 121.3 mm to (405.3, 193.5)
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
Commit message: did some more layout
Parts:
- moved Rfbt5 182.3 mm to (424.9, 256.2), turned to 90 degrees
- moved Rfbb5 181.7 mm to (424.9, 253.1), turned to 90 degrees
- moved Ccomp5 180.2 mm to (426.7, 254.6), turned to 90 degrees
- moved Cramp3 180.1 mm to (427.5, 250.7), turned to 180 degrees
- moved Css3 179.2 mm to (427.5, 252.3), turned to 180 degrees
- moved Cvcc4 179.1 mm to (438.9, 252.7), turned to -90 degrees
- moved Cboot4 178.4 mm to (437.5, 247.9)
- moved Ccomp6 178.0 mm to (428.2, 254.6), turned to 90 degrees
- moved M3 176.4 mm to (444.5, 247.9)
- moved Rcomp3 176.4 mm to (427.5, 256.9), turned to 180 degrees
- moved Cinx4 176.3 mm to (432.0, 247.9)
- moved Cin_2 174.2 mm to (432.0, 243.2)
- moved Rt3 170.6 mm to (427.5, 249.1), turned to 180 degrees
- moved L7 168.7 mm to (436.9, 240.7)
- moved Cin5 166.7 mm to (432.0, 244.8)
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
Commit message: coordinated labels in schem
Labeled all components to be Rxx, Cxx, ext forms through all sheets so labels for BOM and layout are work together as one long list.
Parts:
- added Q13: CSD19538Q3AT, foot:CSD19538Q3AT, F.Cu at (11.0, 2.26)
- added U23: TPS23861PWR, foot:TPS23861PWR, F.Cu at (3.95, 5.17)
- Q8: renamed from Q6; footprint Dependencies:CSD19537Q3 -> foot:CSD19537Q3
- renumbered Cin1 to C15, Cinx1 to C16, Cramp1 to C17, Css1 to C18, Ccomp1 to C19, Ccomp2 to C20, Cboot1 to C21, Cvcc1 to C22, C15 to C23, Cout1 to C24, Cout_1 to C25, Cin2 to C26, Cinx2 to C27, Cvcc2 to C28, Cboot2 to C29, Cout2 to C30, Coutx1 to C31, C16 to C32, Cin3 to C33, Cout3 to C34, C17 to C35, Cin4 to C36, Cinx3 to C37, Cramp2 to C38, Css2 to C39, Ccomp3 to C40, Ccomp4 to C41, Cvcc3 to C42, Cboot3 to C43, C19 to C44, Coutx2 to C45, Coutx3 to C46, Cout4 to C47, C20 to C48, C21 to C49, C22 to C50, C23 to C51, C24 to C52, C25 to C53, C26 to C54, C27 to C55, C28 to C56, C29 to C57, C30 to C58, C31 to C59, C32 to C60, C33 to C61, C34 to C62, C35 to C63, C36 to C64, C37 to C65, C38 to C66, C39 to C67, Cramp3 to C68, Cin5 to C69, Css3 to C70, Cin_1 to C71, Cin_2 to C72, Cinx4 to C73, Ccomp5 to C74, Ccomp6 to C75, Cvcc4 to C76, Cboot4 to C77, Coutx4 to C78, Coutx5 to C79, Cout5 to C80, Cout_2 to C81, C40 to C82, C43 to C83, C42 to C84, C41 to C86, J14 to J13, J15 to J14, Q8 to Q10, M3 to Q11, M4 to Q12, M1 to Q5, M2 to Q6, Q5 to Q7, Q7 to Q9, R14 to R12, R17 to R13, R18 to R14, R19 to R15, R20 to R16, Ruv1 to R17, Ruv2 to R18, Rt1 to R19, Renable1 to R20, Rcomp1 to R21, Rsense1 to R22, Rfbt1 to R23, Rfbb1 to R24, R21 to R25, R22 to R26, Rpgood1 to R27, Rfbt2 to R28, Rfbb2 to R29, R23 to R30, R24 to R31, Rfbt3 to R32, Rfbb3 to R33, R25 to R34, R26 to R35, Ruv3 to R36, Ruv4 to R37, Rramp1 to R38, Rt2 to R39, Rcomp2 to R40, Rfbb4 to R41, Renable2 to R42, Rfbt4 to R43, Rsense2 to R44, R27 to R45, R28 to R46, R29 to R47, R30 to R48, R31 to R49, R32 to R50, R33 to R51, R34 to R52, R35 to R53, R36 to R54, R37 to R55, R38 to R56, R39 to R57, R40 to R58, R41 to R59, R42 to R60, R43 to R61, R44 to R62, Ruv5 to R63, Ruv6 to R64, Renable3 to R65, Rt3 to R66, Rcomp3 to R67, Rfbb5 to R68, Rfbt5 to R69, Rsense3 to R70, R45 to R71, R46 to R72, R48 to R73, R51 to R74, R52 to R75, R50 to R76, R49 to R77, R47 to R78

Commit message: last push before removing oring
i think we're going with an interlock system instead. the battery oring on here will take far too much physical room on the board to make it worthwhile. this push removes the oring and assumes a single power input.
Parts:
- removed J10, J8, J9: XT90PW-M, Connector_AMASS:AMASS_XT90PW-M_1x02_P10.90mm_Horizontal
- J1, R1, R2, R3, R4, R5: moved to B.Cu
- J3: footprint Connector_PinHeader_2.54mm:PinHeader_1x02_P2.54mm_Vertical -> Connector_PinHeader_2.54mm:PinHeader_1x05_P2.54mm_Vertical
- R71: footprint Resistor_SMD:R_Shunt_Vishay_WSR2_WSR3_KelvinConnection -> Resistor_SMD:R_Shunt_Vishay_WSK2512_6332Metric_T2.21mm
- U13, U15, U20, U22, U9: footprint Package_SO:HVSSOP-10-1EP_3x3mm_P0.5mm_EP1.83x1.89mm -> Package_SO:TSSOP-10_3x3mm_P0.5mm
- U16: footprint Dependencies:LM76005RNPR -> Dependencies:RNP0030A
- moved C10 409.4 mm to (94.8, 169.0)
- moved C11 409.4 mm to (82.2, 159.7)
- moved C12 409.4 mm to (95.1, 159.6)
- moved C13 409.4 mm to (92.1, 156.3)
- moved C14 409.4 mm to (92.6, 152.2)
- moved D10 409.4 mm to (91.0, 165.7)
- moved D11 409.4 mm to (85.7, 156.7)
- moved D6 409.4 mm to (81.1, 168.2)
- moved D7 409.4 mm to (81.1, 164.4)
- moved D8 409.4 mm to (78.3, 157.7)
- moved D9 409.4 mm to (74.6, 157.7)
- moved Q1 409.4 mm to (90.5, 168.2)
- moved Q2 409.4 mm to (83.1, 156.0)
- moved Q3 409.4 mm to (92.6, 161.4)
- moved Q4 409.4 mm to (89.4, 157.3)
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Connections:
- C38 pad 1: Net-(U14-RAMP) -> Net-(U14-HB)
- C39 pad 1: Net-(U14-SS) -> unconnected-(C39-Pad1)
- C40 pad 2: Net-(U14-FB) -> Net-(U14-SS)
- C41 pad 1: Net-(U14-COMP) -> Net-(C41-Pad1)
- C41 pad 2: Net-(U14-FB) -> Net-(U14-SS)
- C42 pad 1: Net-(U14-VCC) -> Net-(U14-FB)
- C43 pad 2: Net-(U14-HB) -> unconnected-(C43-Pad2)
- C59 pad 2: Net-(U17-BOOT) -> unconnected-(C59-Pad2)
- C60 pad 1: Net-(U18-VDD) -> Net-(Q9-D)
- C60 pad 2: Net-(U17-FB) -> Net-(C60-Pad2)
- C61 pad 1: Net-(U18-VDD) -> Net-(Q9-D)
- C62 pad 1: Net-(U18-VDD) -> Net-(Q9-D)
- C63 pad 2: Net-(U18-VDD) -> Net-(Q9-D)
- C64 pad 2: Net-(U18-VREG_1V2) -> unconnected-(C64-Pad2)
- C65 pad 2: Net-(U18-VREG_2V7) -> unconnected-(C65-Pad2)
- F5 pad 1: Net-(U18-VBUS_SENSE) -> Net-(Q10-D)
- J11 pad 1: (no net) -> GND
- J11 pad 2: (no net) -> /batt_inA
- J12 pad 1: (no net) -> GND
- J12 pad 2: (no net) -> /batt_inB
- J13 pad A9: Net-(J13-VBUS-PadA9) -> Net-(J13-VBUS-PadA4)
- J13 pad B4: Net-(J13-VBUS-PadA9) -> Net-(J13-VBUS-PadA4)
- J13 pad B5: Net-(J13-CC2) -> unconnected-(J13-CC2-PadB5)
- J13 pad B9: Net-(J13-VBUS-PadA9) -> Net-(J13-VBUS-PadA4)
- J4 pad 1: (no net) -> GND
- J4 pad 2: (no net) -> +5V@4A
- J5 pad 1: (no net) -> GND
- J5 pad 2: (no net) -> +3.3V@1A
- J6 pad 1: (no net) -> GND
- J6 pad 2: (no net) -> 5V@12A
- J7 pad 1: (no net) -> GND
- J7 pad 2: (no net) -> +BATT
- L6 pad 1: Net-(U17-SW) -> unconnected-(L6-Pad1)
- L6 pad 2: Net-(U18-VDD) -> Net-(Q9-D)
- Q10 pad D1: Net-(U18-VBUS_SENSE) -> Net-(Q10-D)
- Q7 pad 4: Net-(U14-HO) -> Net-(U14-VOUT)
- Q8 pad 4: Net-(U14-LO) -> unconnected-(Q8-Pad4)
- Q9 pad D1: Net-(U18-VDD) -> Net-(Q9-D)
- R13 pad 1: Net-(U5-Vss) -> unconnected-(R13-Pad1)
- R14 pad 1: Net-(U6-Vss) -> unconnected-(R14-Pad1)
- R15 pad 2: Net-(U5-IN) -> unconnected-(R15-Pad2)
- R16 pad 2: Net-(U6-IN) -> unconnected-(R16-Pad2)
- R25 pad 2: Net-(U9-Vin+) -> unconnected-(R25-Pad2)
- R25 pad 3: Net-(U9-Vin-) -> unconnected-(R25-Pad3)
- R31 pad 2: Net-(U11-Vin+) -> unconnected-(R31-Pad2)
- R31 pad 3: Net-(U11-Vin-) -> unconnected-(R31-Pad3)
- R35 pad 2: Net-(U13-Vin+) -> unconnected-(R35-Pad2)
- R35 pad 3: Net-(U13-Vin-) -> unconnected-(R35-Pad3)
- R36 pad 2: Net-(U14-UVLO) -> Net-(R36-Pad2)
- R37 pad 1: Net-(U14-UVLO) -> Net-(R36-Pad2)
- R38 pad 1: Net-(U14-VCC) -> Net-(U14-FB)
- R38 pad 2: Net-(U14-RAMP) -> Net-(U14-HB)
- R39 pad 1: Net-(U14-RT) -> unconnected-(R39-Pad1)
- R40 pad 1: Net-(U14-COMP) -> Net-(C41-Pad1)
- R41 pad 1: Net-(U14-FB) -> Net-(U14-SS)
- R42 pad 2: Net-(U14-EN) -> unconnected-(R42-Pad2)
- R43 pad 2: Net-(U14-FB) -> Net-(U14-SS)
- R45 pad 2: Net-(U15-Vin+) -> unconnected-(R45-Pad2)
- R45 pad 3: Net-(U15-Vin-) -> unconnected-(R45-Pad3)
- R50 pad 1: Net-(U17-FB) -> Net-(C60-Pad2)
- R50 pad 2: Net-(U18-VDD) -> Net-(Q9-D)
- R51 pad 1: Net-(U18-GPIO3) -> Net-(R51-Pad1)
- R51 pad 2: Net-(U17-FB) -> Net-(C60-Pad2)
- R52 pad 1: Net-(U18-GPIO2) -> Net-(U18-VCONN)
- R52 pad 2: Net-(U18-GPIO3) -> Net-(R51-Pad1)
- R53 pad 1: Net-(U18-GPIO1) -> Net-(R53-Pad1)
- R53 pad 2: Net-(U18-GPIO2) -> Net-(U18-VCONN)
- R54 pad 1: Net-(U18-GPIO0) -> Net-(U18-RESET)
- R54 pad 2: Net-(U18-GPIO1) -> Net-(R53-Pad1)
- R55 pad 2: Net-(U18-GPIO0) -> Net-(U18-RESET)
- R56 pad 2: Net-(U18-VVAR_ADDR0) -> unconnected-(R56-Pad2)
- R58 pad 1: Net-(U18-VBUS_DISCH) -> Net-(U19-G)
- R58 pad 2: Net-(U18-VDD) -> Net-(Q9-D)
- R60 pad 1: Net-(U18-VBUS_EN_SRC) -> Net-(U18-VDD)
- R61 pad 2: Net-(U20-Vin+) -> unconnected-(R61-Pad2)
- R61 pad 3: Net-(U20-Vin-) -> unconnected-(R61-Pad3)
- R61 pad 4: Net-(J13-VBUS-PadA4) -> Net-(R61-Pad4)
- R62 pad 1: Net-(J13-VBUS-PadA4) -> Net-(R61-Pad4)
- R71 pad 2: Net-(U22-Vin+) -> unconnected-(R71-Pad2)
- TP10 pad 1: Net-(J13-VBUS-PadA4) -> Net-(R61-Pad4)
- U11 pad 10: Net-(U11-Vin+) -> unconnected-(U11-Vin+-Pad10)
- U11 pad 9: Net-(U11-Vin-) -> unconnected-(U11-Vin--Pad9)
- U13 pad 10: Net-(U13-Vin+) -> unconnected-(U13-Vin+-Pad10)
- U13 pad 9: Net-(U13-Vin-) -> unconnected-(U13-Vin--Pad9)
- U14 pad 1: +BATT -> unconnected-(U14-VIN-Pad1)
- U14 pad 10: Net-(D17-K) -> Net-(U14-VOUT)
- U14 pad 12: Net-(D16-A) -> unconnected-(U14-CS-Pad12)
- U14 pad 13: GND -> unconnected-(U14-CSG-Pad13)
- U14 pad 15: Net-(U14-LO) -> unconnected-(U14-LO-Pad15)
- U14 pad 16: Net-(U14-VCC) -> +BATT
- U14 pad 17: GND -> unconnected-(U14-VCCX-Pad17)
- U14 pad 19: Net-(U14-HO) -> Net-(D16-K)
- U14 pad 2: Net-(U14-UVLO) -> unconnected-(U14-UVLO-Pad2)
- U14 pad 20: Net-(D16-K) -> unconnected-(U14-HS-Pad20)
- U14 pad 3: Net-(U14-RT) -> unconnected-(U14-RT-Pad3)
- U14 pad 4: Net-(U14-EN) -> unconnected-(U14-EN-Pad4)
- U14 pad 5: Net-(U14-RAMP) -> Net-(D17-K)
- U14 pad 9: Net-(U14-COMP) -> unconnected-(U14-COMP-Pad9)
- U15 pad 10: Net-(U15-Vin+) -> unconnected-(U15-Vin+-Pad10)
- U15 pad 9: Net-(U15-Vin-) -> unconnected-(U15-Vin--Pad9)
- U17 pad 1: Net-(U17-BOOT) -> unconnected-(U17-BOOT-Pad1)
- U17 pad 3: GND -> unconnected-(U17-*EN1-Pad3)
- U17 pad 4: Net-(U17-FB) -> unconnected-(U17-FB-Pad4)
- U17 pad 5: /USB-C PD/+10VDC -> unconnected-(U17-EN2-Pad5)
- U17 pad 6: GND -> unconnected-(U17-GND-Pad6)
- U17 pad 7: /USB-C PD/+10VDC -> unconnected-(U17-VIN-Pad7)
- U17 pad 8: Net-(U17-SW) -> unconnected-(U17-SW-Pad8)
- U17 pad EPAD: GND -> unconnected-(U17-PadEPAD)
- U18 pad 10: GND -> unconnected-(U18-GND-Pad10)
- U18 pad 11: Net-(U18-GPIO1) -> unconnected-(U18-GPIO1-Pad11)
- U18 pad 12: Net-(U18-GPIO0) -> GND
- U18 pad 13: Net-(U18-VVAR_ADDR0) -> unconnected-(U18-VVAR_ADDR0-Pad13)
- U18 pad 14: Net-(U18-GPIO2) -> Net-(J13-CC1)
- U18 pad 15: Net-(U18-GPIO3) -> unconnected-(U18-GPIO3-Pad15)
- U18 pad 18: Net-(U18-VBUS_SENSE) -> unconnected-(U18-VBUS_SENSE-Pad18)
- U18 pad 19: Net-(U18-VBUS_DISCH) -> unconnected-(U18-VBUS_DISCH-Pad19)
- U18 pad 2: Net-(J13-CC1) -> unconnected-(U18-CC1-Pad2)
- U18 pad 20: Net-(U18-VBUS_EN_SRC) -> unconnected-(U18-VBUS_EN_SRC-Pad20)
- U18 pad 21: Net-(U18-VREG_1V2) -> unconnected-(U18-VREG_1V2-Pad21)
- U18 pad 22: GND -> unconnected-(U18-VSYS-Pad22)
- U18 pad 23: Net-(U18-VREG_2V7) -> unconnected-(U18-VREG_2V7-Pad23)
- U18 pad 25: GND -> unconnected-(U18-EP-Pad25)
- U18 pad 3: GND -> Net-(U18-VCONN)
- U18 pad 4: Net-(J13-CC2) -> unconnected-(U18-CC2-Pad4)
- U18 pad 6: GND -> Net-(U18-RESET)
- U18 pad 7: /USB-C PD/SCL -> unconnected-(U18-SCL-Pad7)
- U18 pad 8: /USB-C PD/SDA -> unconnected-(U18-SDA-Pad8)
- U18 pad 9: unconnected-(U18-ALERT--Pad9) -> /USB-C PD/SCL
- U19 pad 1: Net-(U18-VBUS_DISCH) -> Net-(U19-G)
- U19 pad 2: Net-(U18-VDD) -> Net-(Q9-D)
- U20 pad 10: Net-(U20-Vin+) -> unconnected-(U20-Vin+-Pad10)
- U20 pad 9: Net-(U20-Vin-) -> unconnected-(U20-Vin--Pad9)
- U22 pad 10: Net-(U22-Vin+) -> unconnected-(U22-Vin+-Pad10)
- U22 pad 9: Net-(U22-Vin-) -> unconnected-(U22-Vin--Pad9)
- U5 pad 1: Net-(Q3-D) -> unconnected-(U5-OUT-Pad1)
- U5 pad 2: Net-(D10-K) -> unconnected-(U5-GATE-Pad2)
- U5 pad 4: Net-(U5-IN) -> unconnected-(U5-IN-Pad4)
- U5 pad 5: /PE7 -> unconnected-(U5-~{SHDN}-Pad5)
- U5 pad 6: Net-(U5-Vss) -> unconnected-(U5-Vss-Pad6)
- U5 pad 7: GND -> unconnected-(U5-Pad-Pad7)
- U6 pad 1: Net-(Q3-D) -> unconnected-(U6-OUT-Pad1)
- U6 pad 2: Net-(D11-K) -> unconnected-(U6-GATE-Pad2)
- U6 pad 4: Net-(U6-IN) -> unconnected-(U6-IN-Pad4)
- U6 pad 5: /PE8 -> unconnected-(U6-~{SHDN}-Pad5)
- U6 pad 6: Net-(U6-Vss) -> unconnected-(U6-Vss-Pad6)
- U6 pad 7: GND -> unconnected-(U6-Pad-Pad7)
- U9 pad 10: Net-(U9-Vin+) -> unconnected-(U9-Vin+-Pad10)
- U9 pad 9: Net-(U9-Vin-) -> unconnected-(U9-Vin--Pad9)
Routing:
- net GND: track 1.23 -> 45.7 mm, vias 0 -> 20
- net +3.3V: track 0.00 -> 27.9 mm, vias 0 -> 14
- net (no net): track 0.00 -> 19.1 mm, vias 0 -> 2
- net /PC10: track 0.00 -> 15.6 mm, vias 0 -> 1
- net /PC11: track 0.00 -> 14.5 mm, vias 0 -> 3
- net /SWDIO: track 0.00 -> 13.3 mm, vias 0 -> 1
- net /PD2: track 0.00 -> 12.6 mm, vias 0 -> 3
- net Net-(U18-GPIO0): track 12.3 -> 0.00 mm, vias 2 -> 0
- net Net-(U18-GPIO1): track 11.6 -> 0.00 mm, vias 2 -> 0
- net /PC8: track 0.00 -> 11.1 mm, vias 0 -> 1
- net /PC12: track 0.00 -> 10.9 mm, vias 0 -> 1
- net /SWO/TRACE: track 0.00 -> 10.5 mm
- net /SWCLK: track 0.00 -> 9.98 mm, vias 0 -> 2
- net Net-(U18-GPIO2): track 9.24 -> 0.00 mm, vias 2 -> 0
- net Net-(J13-CC1): track 0.00 -> 9.24 mm, vias 0 -> 2
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- added copper zone on In3.Cu, net +3.3V
- added copper zone on In1.Cu, net GND
Other:
- copper layers 2 -> 6

Commit message: did lots of routing
Parts:
- removed C10, C11: 470nF, Capacitor_SMD:C_0603_1608Metric
- removed C12, C13: 1.5uF, Capacitor_SMD:C_0603_1608Metric
- removed D10, D11: DDZ9699T 12V, Diode_SMD:D_SOD-523
- removed D6, D7, D8, D9: SMAJ64A, Diode_SMD:D_SMA
- removed J12: XT90PW-M, Connector_AMASS:AMASS_XT90PW-M_1x02_P10.90mm_Horizontal
- removed Q1, Q2: IPT012N08N5, Package_TO_SOT_SMD:SOT-23
- removed Q3, Q4: BSC093N15NS5, Package_TO_SOT_SMD:SOT-23
- removed R13, R14: 1k, Resistor_SMD:R_0603_1608Metric_Pad0.98x0.95mm_HandSolder
- removed R15, R16: 100k, Resistor_SMD:R_0603_1608Metric_Pad0.98x0.95mm_HandSolder
- removed TP3, TP4: TestPoint, TestPoint:TestPoint_Pad_D2.0mm
- removed U5, U6: LTC4359-DCB, Package_DFN_QFN:DFN-6-1EP_3x2mm_P0.5mm_EP1.65x1.35mm
- U16: footprint Dependencies:RNP0030A -> Dependencies:LM76005RNPR
- U20: footprint Package_SO:TSSOP-10_3x3mm_P0.5mm -> Package_SO:HVSSOP-10-1EP_3x3mm_P0.5mm_EP1.83x1.89mm
- moved C35 437.7 mm to (111.9, 83.0), turned to 90 degrees
- moved L3 436.7 mm to (105.9, 87.6), turned to 90 degrees
- moved F3 436.1 mm to (109.6, 85.7), turned to 180 degrees
- moved R33 435.1 mm to (101.9, 91.8), turned to 90 degrees
- moved C34 434.0 mm to (108.1, 88.5), turned to -90 degrees
- moved R32 433.7 mm to (103.6, 91.8), turned to -90 degrees
- moved U13 432.4 mm to (115.9, 84.8), turned to 180 degrees
- moved U12 432.1 mm to (105.4, 91.9), turned to 90 degrees
- moved C33 430.6 mm to (107.4, 91.9), turned to 90 degrees
- moved R35 429.4 mm to (113.4, 88.9), turned to 0 degrees
- moved D15 424.7 mm to (113.7, 92.7), turned to 90 degrees
- moved R34 423.8 mm to (116.3, 91.7), turned to 180 degrees
- moved TP8 420.8 mm to (119.7, 92.1), turned to 180 degrees
- moved C32 370.1 mm to (103.4, 113.3), turned to 90 degrees
- moved U11 364.5 mm to (105.7, 109.9), turned to 90 degrees
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Connections:
- C35 pad 2: /3V3@1A/+3.3V -> +3.3V
- C59 pad 2: unconnected-(C59-Pad2) -> Net-(U17-BOOT)
- C60 pad 2: Net-(C60-Pad2) -> Net-(U17-FB)
- C64 pad 2: unconnected-(C64-Pad2) -> Net-(U18-VREG_1V2)
- C65 pad 2: unconnected-(C65-Pad2) -> Net-(U18-VREG_2V7)
- J11 pad 2: /batt_inA -> +BATT
- J13 pad A9: Net-(J13-VBUS-PadA4) -> Net-(J13-VBUS-PadA9)
- J13 pad B4: Net-(J13-VBUS-PadA4) -> Net-(J13-VBUS-PadA9)
- J13 pad B5: unconnected-(J13-CC2-PadB5) -> Net-(J13-CC2)
- J13 pad B9: Net-(J13-VBUS-PadA4) -> Net-(J13-VBUS-PadA9)
- J5 pad 2: +3.3V@1A -> +3.3V
- L6 pad 1: unconnected-(L6-Pad1) -> Net-(U17-SW)
- R34 pad 1: +3.3V@1A -> +3.3V
- R35 pad 4: +3.3V@1A -> +3.3V
- R50 pad 1: Net-(C60-Pad2) -> Net-(U17-FB)
- R51 pad 1: Net-(R51-Pad1) -> Net-(U18-GPIO3)
- R51 pad 2: Net-(C60-Pad2) -> Net-(U17-FB)
- R52 pad 1: Net-(U18-VCONN) -> Net-(U18-GPIO2)
- R52 pad 2: Net-(R51-Pad1) -> Net-(U18-GPIO3)
- R53 pad 1: Net-(R53-Pad1) -> Net-(U18-GPIO1)
- R53 pad 2: Net-(U18-VCONN) -> Net-(U18-GPIO2)
- R54 pad 1: Net-(U18-RESET) -> Net-(U18-GPIO0)
- R54 pad 2: Net-(R53-Pad1) -> Net-(U18-GPIO1)
- R55 pad 2: Net-(U18-RESET) -> Net-(U18-GPIO0)
- R56 pad 2: unconnected-(R56-Pad2) -> Net-(U18-VVAR_ADDR0)
- R58 pad 1: Net-(U19-G) -> Net-(U18-VBUS_DISCH)
- R60 pad 1: Net-(U18-VDD) -> Net-(U18-VBUS_EN_SRC)
- R61 pad 2: unconnected-(R61-Pad2) -> Net-(U20-Vin+)
- R61 pad 3: unconnected-(R61-Pad3) -> Net-(U20-Vin-)
- R61 pad 4: Net-(R61-Pad4) -> Net-(J13-VBUS-PadA4)
- R62 pad 1: Net-(R61-Pad4) -> Net-(J13-VBUS-PadA4)
- TP10 pad 1: Net-(R61-Pad4) -> Net-(J13-VBUS-PadA4)
- TP8 pad 1: +3.3V@1A -> +3.3V
- U13 pad 2: /3V3@1A/+3.3V -> +3.3V
- U13 pad 6: /3V3@1A/+3.3V -> +3.3V
- U16 pad 36: (no net) -> GND
- U16 pad 38: (no net) -> GND
- U16 pad 39: (no net) -> GND
- U16 pad 40: (no net) -> GND
- U16 pad 41: (no net) -> GND
- U17 pad 1: unconnected-(U17-BOOT-Pad1) -> Net-(U17-BOOT)
- U17 pad 3: unconnected-(U17-*EN1-Pad3) -> GND
- U17 pad 4: unconnected-(U17-FB-Pad4) -> Net-(U17-FB)
- U17 pad 5: unconnected-(U17-EN2-Pad5) -> /USB-C PD/+10VDC
- U17 pad 6: unconnected-(U17-GND-Pad6) -> GND
- U17 pad 7: unconnected-(U17-VIN-Pad7) -> /USB-C PD/+10VDC
- U17 pad 8: unconnected-(U17-SW-Pad8) -> Net-(U17-SW)
- U17 pad EPAD: unconnected-(U17-PadEPAD) -> GND
- U18 pad 10: unconnected-(U18-GND-Pad10) -> GND
- U18 pad 11: unconnected-(U18-GPIO1-Pad11) -> Net-(U18-GPIO1)
- U18 pad 12: GND -> Net-(U18-GPIO0)
- U18 pad 13: unconnected-(U18-VVAR_ADDR0-Pad13) -> Net-(U18-VVAR_ADDR0)
- U18 pad 14: Net-(J13-CC1) -> Net-(U18-GPIO2)
- U18 pad 15: unconnected-(U18-GPIO3-Pad15) -> Net-(U18-GPIO3)
- U18 pad 18: unconnected-(U18-VBUS_SENSE-Pad18) -> Net-(Q10-D)
- U18 pad 19: unconnected-(U18-VBUS_DISCH-Pad19) -> Net-(U18-VBUS_DISCH)
- U18 pad 2: unconnected-(U18-CC1-Pad2) -> Net-(J13-CC1)
- U18 pad 20: unconnected-(U18-VBUS_EN_SRC-Pad20) -> Net-(U18-VBUS_EN_SRC)
- U18 pad 21: unconnected-(U18-VREG_1V2-Pad21) -> Net-(U18-VREG_1V2)
- U18 pad 22: unconnected-(U18-VSYS-Pad22) -> GND
- U18 pad 23: unconnected-(U18-VREG_2V7-Pad23) -> Net-(U18-VREG_2V7)
- U18 pad 24: Net-(U18-VDD) -> Net-(Q9-D)
- U18 pad 25: unconnected-(U18-EP-Pad25) -> GND
- U18 pad 3: Net-(U18-VCONN) -> GND
- U18 pad 4: unconnected-(U18-CC2-Pad4) -> Net-(J13-CC2)
- U18 pad 6: Net-(U18-RESET) -> GND
- U18 pad 7: unconnected-(U18-SCL-Pad7) -> /USB-C PD/SCL
- U18 pad 8: unconnected-(U18-SDA-Pad8) -> /USB-C PD/SDA
- U18 pad 9: /USB-C PD/SCL -> unconnected-(U18-ALERT--Pad9)
- U19 pad 1: Net-(U19-G) -> Net-(U18-VBUS_DISCH)
- U20 pad 10: unconnected-(U20-Vin+-Pad10) -> Net-(U20-Vin+)
- U20 pad 9: unconnected-(U20-Vin--Pad9) -> Net-(U20-Vin-)
- U7 pad 1: Net-(Q3-D) -> +BATT
- U7 pad 2: Net-(Q3-D) -> +BATT
Routing:
- net GND: track 45.7 -> 107.7 mm, vias 20 -> 36
- net /PC0: track 0.00 -> 47.7 mm, vias 0 -> 2
- net +BATT: track 3.04 -> 42.9 mm
- net +5V@4A: track 0.00 -> 26.8 mm
- net +3.3V: track 27.9 -> 45.8 mm, vias 14 -> 22
- net /USB-C PD/+10VDC: track 0.00 -> 15.7 mm
- net Net-(C30-Pad1): track 0.00 -> 14.6 mm, vias 0 -> 2
- net /5V@4A/+3.3V: track 0.00 -> 13.5 mm, vias 0 -> 3
- net Net-(U18-GPIO0): track 0.00 -> 12.3 mm, vias 0 -> 2
- net Net-(U18-GPIO1): track 0.00 -> 11.6 mm, vias 0 -> 2
- net Net-(C34-Pad1): track 0.00 -> 10.3 mm
- net Net-(U11-Vbus): track 0.00 -> 10.0 mm
- net (no net): track 19.1 -> 28.4 mm
- net Net-(J13-CC1): track 9.24 -> 0.00 mm, vias 2 -> 0
- net Net-(U18-GPIO2): track 0.00 -> 9.24 mm, vias 0 -> 2
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- added copper zone on F.Cu, net +3.3V
- added copper zone on F.Cu, net +BATT
- added copper zone on F.Cu, net GND
- added copper zone on F.Cu, net unconnected-(U11-Vin--Pad9)
